File: HVPS_SMD/HVPS_SMD.sch (KiCad schematic (older format))
At the start: 20 parts, among them J1 CONN_01X02, J2 CONN_01X02, J3 CONN_01X02, Q1 AO4294, T1 WE-FLEX_ER11_5, U1 LM3478SOIC8

Commit message: Fixed external footprint references
Parts:
- C1, C3: footprint Capacitors_SMD:C_1210 -> lib_fp:C_1210
- C2, Cc1, Cs1: footprint Capacitors_SMD:C_0603 -> lib_fp:C_0603
- D1: footprint nixiemisc:nixiemisc-DO-219AB -> lib_fp:nixiemisc-DO-219AB
- J1, J2, J3: footprint SparkFun-Connectors:SparkFun-Connectors-1X02_NO_SILK -> lib_fp:SparkFun-Connectors-1X02_NO_SILK
- Q1: footprint nixiemisc:nixiemisc-SO08 -> lib_fp:nixiemisc-SO08
- R1, R2, Rc1, Rf1: footprint Resistors_SMD:R_0805 -> lib_fp:R_0805
- R3, R4: footprint Resistors_SMD:R_0603 -> lib_fp:R_0603
- Rs1: footprint Resistors_SMD:R_1206 -> lib_fp:R_1206
- Rsen1: footprint Resistors_SMD:R_2010 -> lib_fp:R_2010
- T1: footprint nixiemisc:nixiemisc-WE-FLEX_ER11_5 -> lib_fp:nixiemisc-WE-FLEX_ER11_5
- U1: footprint nixiemisc:nixiemisc-SOIC8 -> lib_fp:nixiemisc-SOIC8
Changed lines of the file:
@@
 F 0 "U1" H 3800 3825 45  0000 L BNN
 F 1 "LM3478SOIC8" H 4400 3000 45  0000 L BNN
-F 2 "nixiemisc:nixiemisc-SOIC8" H 4330 3650 20  0001 C CNN
+F 2 "lib_fp:nixiemisc-SOIC8" H 4330 3650 20  0001 C CNN
 F 3 "" H 4300 3500 60  0001 C CNN
 	1    4300 3500
@@
 F 0 "T1" H 6400 2500 45  0000 L BNN
 F 1 "WE-FLEX_ER11_5" H 6400 1500 45  0000 L BNN
-F 2 "nixiemisc:nixiemisc-WE-FLEX_ER11_5" H 6680 2150 20  0001 C CNN
+F 2 "lib_fp:nixiemisc-WE-FLEX_ER11_5" H 6680 2150 20  0001 C CNN
 F 3 "" H 6650 2000 60  0001 C CNN
 	1    6650 2000
@@
 F 0 "Q1" H 5750 3325 45  0000 L BNN
 F 1 "AO4294" H 5750 3250 45  0000 L BNN
-F 2 "nixiemisc:nixiemisc-SO08" H 5580 3450 20  0001 C CNN
+F 2 "lib_fp:nixiemisc-SO08" H 5580 3450 20  0001 C CNN
 F 3 "" H 5550 3300 60  0001 C CNN
 	1    5550 3300
@@
 F 0 "Rsen1" H 5680 4070 50  0000 L CNN
 F 1 "0.06" H 5680 4010 50  0000 L CNN
-F 2 "Resistors_SMD:R_2010" H 5650 4050 50  0001 C CNN
+F 2 "lib_fp:R_2010" H 5650 4050 50  0001 C CNN
 F 3 "" H 5650 4050 50  0001 C CNN
 	1    5650 4050
@@
 F 0 "C2" H 5410 4120 50  0000 L CNN
 F 1 "0.01uF" H 5410 3970 50  0000 L CNN
-F 2 "Capacitors_SMD:C_0603" H 5400 4050 50  0001 C CNN
+F 2 "lib_fp:C_0603" H 5400 4050 50  0001 C CNN
 F 3 "" H 5400 4050 50  0001 C CNN
 	1    5400 4050
@@
 F 0 "Cc1" H 3460 3970 50  0000 L CNN
 F 1 "22nF" H 3460 3820 50  0000 L CNN
-F 2 "Capacitors_SMD:C_0603" H 3450 3900 50  0001 C CNN
+F 2 "lib_fp:C_0603" H 3450 3900 50  0001 C CNN
 F 3 "" H 3450 3900 50  0001 C CNN
 	1    3450 3900
@@
 F 0 "Rc1" H 3480 4170 50  0000 L CNN
 F 1 "4.7k" H 3480 4110 50  0000 L CNN
-F 2 "Resistors_SMD:R_0805" H 3450 4150 50  0001 C CNN
+F 2 "lib_fp:R_0805" H 3450 4150 50  0001 C CNN
 F 3 "" H 3450 4150 50  0001 C CNN
 	1    3450 4150
@@
 F 0 "C3" H 7560 1670 50  0000 L CNN
 F 1 "0.22uF" H 7560 1520 50  0000 L CNN
-F 2 "Capacitors_SMD:C_1210" H 7550 1600 50  0001 C CNN
+F 2 "lib_fp:C_1210" H 7550 1600 50  0001 C CNN
 F 3 "" H 7550 1600 50  0001 C CNN
 	1    7550 1600
@@
 F 0 "R2" H 7030 3270 50  0000 L CNN
 F 1 "604k" H 7030 3210 50  0000 L CNN
-F 2 "Resistors_SMD:R_0805" H 7000 3250 50  0001 C CNN
+F 2 "lib_fp:R_0805" H 7000 3250 50  0001 C CNN
 F 3 "" H 7000 3250 50  0001 C CNN
 	1    7000 3250
@@
 F 0 "R3" H 7030 4020 50  0000 L CNN
 F 1 "10.2k" H 7030 3960 50  0000 L CNN
-F 2 "Resistors_SMD:R_0603" H 7000 4000 50  0001 C CNN
+F 2 "lib_fp:R_0603" H 7000 4000 50  0001 C CNN
 F 3 "" H 7000 4000 50  0001 C CNN
 	1    7000 4000
@@
 F 0 "R4" H 7480 3420 50  0000 L CNN
 F 1 "30k" H 7480 3360 50  0000 L CNN
-F 2 "Resistors_SMD:R_0603" H 7450 3400 50  0001 C CNN
+F 2 "lib_fp:R_0603" H 7450 3400 50  0001 C CNN
 F 3 "" H 7450 3400 50  0001 C CNN
 	1    7450 3400
@@
 F 0 "Rf1" H 3480 3420 50  0000 L CNN
 F 1 "47k" H 3480 3360 50  0000 L CNN
-F 2 "Resistors_SMD:R_0805" H 3450 3400 50  0001 C CNN
+F 2 "lib_fp:R_0805" H 3450 3400 50  0001 C CNN
 F 3 "" H 3450 3400 50  0001 C CNN
 	1    3450 3400
@@
 F 0 "Rs1" H 5180 2770 50  0000 L CNN
 F 1 "249" H 5180 2710 50  0000 L CNN
-F 2 "Resistors_SMD:R_1206" H 5150 2750 50  0001 C CNN
+F 2 "lib_fp:R_1206" H 5150 2750 50  0001 C CNN
 F 3 "" H 5150 2750 50  0001 C CNN
 	1    5150 2750
@@
 F 0 "Cs1" H 5160 2470 50  0000 L CNN
 F 1 "360pF" H 5160 2320 50  0000 L CNN
-F 2 "Capacitors_SMD:C_0603" H 5150 2400 50  0001 C CNN
+F 2 "lib_fp:C_0603" H 5150 2400 50  0001 C CNN
 F 3 "" H 5150 2400 50  0001 C CNN
 	1    5150 2400
@@
 F 0 "C1" H 2725 3550 50  0000 L CNN
 F 1 "100uF" H 2725 3350 50  0000 L CNN
-F 2 "Capacitors_SMD:C_1210" H 2700 3450 50  0001 C CNN
+F 2 "lib_fp:C_1210" H 2700 3450 50  0001 C CNN
 F 3 "" H 2700 3450 50  0001 C CNN
 	1    2700 3450
@@
 F 0 "J2" H 1700 2500 50  0000 C CNN
 F 1 "CONN_01X02" V 1800 2350 50  0000 C CNN
-F 2 "SparkFun-Connectors:SparkFun-Connectors-1X02_NO_SILK" H 1700 2350 50  0001 C CNN
+F 2 "lib_fp:SparkFun-Connectors-1X02_NO_SILK" H 1700 2350 50  0001 C CNN
 F 3 "" H 1700 2350 50  0001 C CNN
 	1    1700 2350
@@
 F 0 "R1" H 7030 3020 50  0000 L CNN
 F 1 "604k" H 7030 2960 50  0000 L CNN
-F 2 "Resistors_SMD:R_0805" H 7000 3000 50  0001 C CNN
+F 2 "lib_fp:R_0805" H 7000 3000 50  0001 C CNN
 F 3 "" H 7000 3000 50  0001 C CNN
 	1    7000 3000
@@
 F 0 "D1" H 7259 1504 45  0000 L BNN
 F 1 "ES1FL R3G" H 7249 1223 45  0000 L BNN
-F 2 "nixiemisc:nixiemisc-DO-219AB" H 7380 1550 20  0001 C CNN
+F 2 "lib_fp:nixiemisc-DO-219AB" H 7380 1550 20  0001 C CNN
 F 3 "" H 7350 1400 60  0001 C CNN
 	1    7350 1400
@@
 F 0 "J1" H 1700 1850 50  0000 C CNN
 F 1 "CONN_01X02" V 1800 1700 50  0000 C CNN
-F 2 "SparkFun-Connectors:SparkFun-Connectors-1X02_NO_SILK" H 1700 1700 50  0001 C CNN
+F 2 "lib_fp:SparkFun-Connectors-1X02_NO_SILK" H 1700 1700 50  0001 C CNN
 F 3 "" H 1700 1700 50  0001 C CNN
 	1    1700 1700
@@
 F 0 "J3" H 2850 2300 50  0000 C CNN
 F 1 "CONN_01X02" V 2950 2150 50  0000 C CNN
-F 2 "SparkFun-Connectors:SparkFun-Connectors-1X02_NO_SILK" H 2850 2150 50  0001 C CNN
+F 2 "lib_fp:SparkFun-Connectors-1X02_NO_SILK" H 2850 2150 50  0001 C CNN
 F 3 "" H 2850 2150 50  0001 C CNN
 	1    2850 2150
